Commit message: add debug points

File: robots/fr3_with_camera.urdf (robot description, URDF)
Before this commit: robot fr3, 14 links, 13 joints
Links:
- link camera: geometry visual mesh filename=package://robots/meshes/visual/d435i_rot4.obj
Joints:
- joint fr3_hand_camera_joint: origin xyz=0.05 0.0 0.05 rpy=1.570796 0.0 -1.570796 -> xyz=0.05 0.0 0.05 rpy=0.0 0.0 1.5707963267948966

Commit message: simulation freezes

File: robots/fr3_with_camera.urdf (robot description, URDF)
Before this commit: robot fr3, 14 links, 13 joints
Links:
- link camera: geometry visual mesh filename=package://robots/meshes/visual/d435i_rot.obj
Joints:
- joint fr3_hand_camera_joint: origin xyz=0.05 0.0 0.05 rpy=0.0 0.0 1.5707963267948966 -> xyz=0.05 0.0 0.05 rpy=0.0 -0.01 1.57

Commit message: comment out visual of the camera

File: robots/fr3_with_camera.urdf (robot description, URDF)
Before this commit: robot fr3, 14 links, 13 joints
Links:
- link camera: geometry 
Joints:
- joint fr3_hand_camera_joint: origin xyz=0.05 0.0 0.05 rpy=0.0 -0.01 1.57 -> xyz=0.05 0.0 0.05 rpy=0.0 0.0 1.57

Commit message: Put camera visual model back

File: robots/fr3_with_camera.urdf (robot description, URDF)
Before this commit: robot fr3, 14 links, 13 joints
Links:
- link camera: geometry visual mesh filename=package://robots/meshes/visual/d435i_reduced.obj
