Commit message: add second board

File: robots/apriltag_id1.urdf (robot description, URDF)
Before this commit: robot mesh, 1 links, 0 joints
Links:
- link baselink: geometry collision mesh filename=package://robots/meshes/visual/apriltag_id1.obj scale=1 1 1; visual mesh filename=package://robots/meshes/visual/apriltag_id1.obj scale=1 1 1
