Commit message: updated urdf models

File: robots/box_small.urdf (robot description, URDF)
Before this commit: robot box, 1 links, 0 joints
Links:
- removed link baselink
- added link link1, mass .0; visual box size=0.2 0.6 0.005
- added link link2, mass .0; visual cylinder length=0.25 radius=0.005; visual cylinder length=0.25 radius=0.005
Joints:
- added joint fixed_joint: type fixed, parent link1, child link2, origin xyz=0 0 0 rpy=0 0 0

File: robots/square1.urdf (robot description, URDF)
Before this commit: robot box, 1 links, 0 joints
Links:
- removed link baselink
- added link link1, mass .0; visual box size=0.10 0.10 0.005
- added link link2, mass .0; visual cylinder length=0.3 radius=0.005
Joints:
- added joint fixed_joint: type fixed, parent link1, child link2, origin xyz=0 0 0 rpy=0 0 0
