Commit message: changed robot urdf

File: robots/fr3_with_bounding_boxes.urdf (robot description, URDF)
Before this commit: robot fr3, 14 links, 13 joints
Links:
- removed link camera
- added link fr3_camera, mass 0.072; visual mesh filename=package://robots/meshes/visual/d435i_reduced.obj
- added link fr3_hand_bounding_box, mass 1e-10
- added link fr3_link3_bounding_box, mass 1e-10
- added link fr3_link4_bounding_box, mass 1e-10
- added link fr3_link5_1_bounding_box, mass 1e-10
- added link fr3_link5_2_bounding_box, mass 1e-10
- added link fr3_link6_bounding_box, mass 1e-10
- added link fr3_link7_bounding_box, mass 1e-10
Joints:
- added joint fr3_hand_bounding_box_joint: type fixed, parent fr3_hand, child fr3_hand_bounding_box, origin xyz=0 0.00 0.02 rpy=0 0 0
- added joint fr3_joint3_bounding_box: type fixed, parent fr3_link3, child fr3_link3_bounding_box, origin xyz=0 0 -0.145 rpy=0 0 0
- added joint fr3_joint4_bounding_box: type fixed, parent fr3_link4, child fr3_link4_bounding_box, origin xyz=0 0 0 rpy=0 0 0
- added joint fr3_joint5_1_bounding_box: type fixed, parent fr3_link5, child fr3_link5_1_bounding_box, origin xyz=0 0 -0.26 rpy=0 0 0
- added joint fr3_joint5_2_bounding_box: type fixed, parent fr3_link5, child fr3_link5_2_bounding_box, origin xyz=0 0.08 -0.13 rpy=0 0 0
- added joint fr3_joint6_bounding_box: type fixed, parent fr3_link6, child fr3_link6_bounding_box, origin xyz=0 0.00 -0.03 rpy=0 0 0
- added joint fr3_joint7_bounding_box: type fixed, parent fr3_link7, child fr3_link7_bounding_box, origin xyz=0 0.00 0.01 rpy=0 0 0
- joint fr3_hand_camera_joint: child camera -> fr3_camera
